File: moirePCB/moirePCB.kicad_sch (KiCad schematic)
At the start: 13 parts, among them U1 ATmega328P-A, U2 BQ24075RGT

Commit message: programmer header
Parts:
- added AE1: T1-915M Antenna, symbol Device:Antenna
- added J1: AVR-ISP-6, symbol Connector:AVR-ISP-6
- added U3: UA78M33, symbol Regulator_Linear:uA7805
- added U4: RFM95W-915S2, symbol RF_Module:RFM95W-915S2
- U2: desc (none) -> Battery Charger
Connections:
- net GND: now also J1.6 (GND), U3.2 (GND), U4.1 (GND), U4.10 (GND), U4.8 (GND)
- net VCC: now also J1.2 (VCC), U3.3 (OUT), U4.13 (3.3V)
- net at C3.2, D1.2 (A), D2.2 (A)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: now also U3.1 (IN)
- net at U1.15 (PB3): now also J1.4 (MOSI)
- net at U1.16 (PB4): now also J1.1 (MISO)
- net at U1.17 (PB5): now also J1.3 (SCK)
- net at U1.29 (~{RESET}/PC6): now also J1.5 (~{RST})
- new net: AE1.1 (A), U4.9 (ANT)

Commit message: esp32 and crystal
Parts:
- removed J1: AVR-ISP-6, symbol Connector:AVR-ISP-6
- removed U1: ATmega328P-A, Package_QFP:TQFP-32_7x7mm_P0.8mm, symbol MCU_Microchip_ATmega:ATmega328P-A
- added C5, C6: 10p, symbol Device:C
- added U1: ESP32-WROOM-32U, RF_Module:ESP32-WROOM-32U, symbol RF_Module:ESP32-WROOM-32U
- added Y1: Crystal_GND24, symbol Device:Crystal_GND24
Connections:
- net GND: now also C5.1, C5.2, C6.1, C6.2, U1.1 (GND), U1.15 (GND), U1.29 (IO5), U1.30 (IO18), U1.38 (GND), U1.39 (GND), Y1.1, Y1.2, Y1.3, Y1.4
- net VCC: now also U1.2 (VDD)
Other:
- moved on the sheet: AE1, U4

Commit message: new esp
Parts:
- removed U1: ESP32-WROOM-32U, RF_Module:ESP32-WROOM-32U, symbol RF_Module:ESP32-WROOM-32U
- removed Y1: Crystal_GND24, symbol Device:Crystal_GND24
- added U1: ESP32-PICO-D4, Package_DFN_QFN:QFN-48-1EP_7x7mm_P0.5mm_EP5.3x5.3mm, symbol RF_Module:ESP32-PICO-D4
- added Y2: 32.768kHz, symbol Device:Crystal
- C1: value 100n -> .1u
- C2: value 10u -> 12pF/50V
- C5: value 10p -> 10u
- C6: value 10p -> 12pF/50V
Connections:
- net GND: now also C2.1, U1.49 (GND); no longer C2.2, C5.1, C6.1
- net VCC: now also C5.1, U1.1 (VDDA), U1.19 (VDD3P3_RTC), U1.3 (VDDA3P3), U1.37 (VDD3P3_CPU), U1.4 (VDDA3P3), U1.43 (VDDA), U1.46 (VDDA); no longer C2.1
- new net: C2.2, U1.12 (IO32), Y2.2
- new net: C6.1, U1.13 (IO33), Y2.1
Other:
- note added: "external RTC crystal"
- moved on the sheet: AE1, BT1, C3, C4, D1, D2, R1, R2, R3, SC1, U2, U3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

Commit message: usb otg
Parts:
- added C7: 100nF, symbol Device:C
- added J1: USB_C_Receptacle, symbol Connector:USB_C_Receptacle
- added R4: 10k, symbol Device:R
- added R6: 5.1k, symbol Device:R
- added R7: 4.7k, symbol Device:R
- added SW1: SW_Push_SPDT, symbol Switch:SW_Push_SPDT
- added SW3: SW_DPDT_x2, symbol Switch:SW_DPDT_x2
- added U5: CH340E, Package_SO:MSOP-10_3x3mm_P0.5mm, symbol Interface_USB:CH340E
Connections:
- net GND: now also C7.2, J1.A1 (GND), J1.A12 (GND), J1.B1 (GND), J1.B12 (GND), J1.S1 (SHIELD), SW1.2 (B), U5.3 (GND)
- net VCC: now also C7.1, R4.2, U5.10 (V3), U5.7 (VCC)
- net at C4.2, U2.13 (IN): now also SW3.2 (B); no longer SC1.1 (+)
- net IO0: now reaches U1.23 (IO0)
- net IO0: now also R7.2, U5.6 (TNOW)
- net RX: now reaches U1.40 (U0RXD/IO3)
- net RX: now also U5.9 (RXD)
- net TX: now reaches U1.41 (U0TXD/IO1)
- net TX: now also U5.8 (TXD)
- net EN: now reaches U1.9 (EN)
- net EN: now also R4.1, SW1.3 (C), U5.4 (~{RTS})
- new net: SC1.1 (+), SW3.1 (A)
- new net: R7.1, U5.5 (~{CTS})
- new net: J1.B5 (CC2), R6.1
- new net: J1.A5 (CC1), R6.2
- new net D+: J1.A6 (D+), J1.B6 (D+), U5.1 (UD+)
- new net D-: J1.A7 (D-), J1.B7 (D-), U5.2 (UD-)
- new net USB5V: J1.A4 (VBUS), J1.A9 (VBUS), J1.B4 (VBUS), J1.B9 (VBUS), SW3.3 (C)
- no-connect marks 0 -> 16
Other:
- note added: "For internal flash use"
- note added: "reset button"
- moved on the sheet: C2, C6, SC1, Y2

Commit message: initial placements
Parts:
- C1, C2, C3, C4, C5, C6, C7: footprint (none) -> Capacitor_SMD:C_0805_2012Metric
- D1, D2, SC1: footprint (none) -> LED_SMD:LED_0805_2012Metric
- J1: footprint (none) -> Connector_USB:USB_C_Receptacle_JAE_DX07S016JA1R1500
- R1, R2, R3, R4, R6, R7: footprint (none) -> Resistor_SMD:R_0805_2012Metric
- SW1: footprint (none) -> Button_Switch_SMD:Panasonic_EVQPUL_EVQPUC
- SW3: footprint (none) -> Button_Switch_SMD:SW_SPDT_PCM12
- U3: footprint (none) -> Package_TO_SOT_SMD:SOT-223-3_TabPin2
- U4: footprint (none) -> RF_Module:HOPERF_RFM9XW_SMD
- Y2: footprint (none) -> Crystal:Crystal_SMD_MicroCrystal_CM9V-T1A-2Pin_1.6x1.0mm
Changed lines of the file:
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@@
       (effects (font (size 1.27 1.27)) (justify left))
     )
-    (property "Footprint" "" (at 33.02 149.606 90)
+    (property "Footprint" "LED_SMD:LED_0805_2012Metric" (at 33.02 149.606 90)
       (effects (font (size 1.27 1.27)) hide)
     )
@@
       (effects (font (size 1.27 1.27)) (justify right))
     )
-    (property "Footprint" "" (at 91.44 175.26 0)
+    (property "Footprint" "LED_SMD:LED_0805_2012Metric" (at 91.44 175.26 0)
       (effects (font (size 1.27 1.27)) hide)
     )
@@
       (effects (font (size 1.27 1.27)) (justify left))
     )
-    (property "Footprint" "" (at 45.4152 138.43 0)
+    (property "Footprint" "Capacitor_SMD:C_0805_2012Metric" (at 45.4152 138.43 0)
       (effects (font (size 1.27 1.27)) hide)
     )
@@
       (effects (font (size 1.27 1.27)) (justify left))
     )
-    (property "Footprint" "" (at 231.902 77.47 90)
+    (property "Footprint" "Resistor_SMD:R_0805_2012Metric" (at 231.902 77.47 90)
       (effects (font (size 1.27 1.27)) hide)
     )
@@
       (effects (font (size 1.27 1.27)))
     )
-    (property "Footprint" "" (at 223.52 140.6652 0)
+    (property "Footprint" "Capacitor_SMD:C_0805_2012Metric" (at 223.52 140.6652 0)
       (effects (font (size 1.27 1.27)) hide)
     )
@@
       (effects (font (size 1.27 1.27)))
     )
-    (property "Footprint" "" (at 38.1 138.43 0)
+    (property "Footprint" "Button_Switch_SMD:SW_SPDT_PCM12" (at 38.1 138.43 0)
       (effects (font (size 1.27 1.27)) hide)
     )
@@
       (effects (font (size 1.27 1.27)) (justify left))
     )
-    (property "Footprint" "" (at 116.5352 41.91 0)
+    (property "Footprint" "Capacitor_SMD:C_0805_2012Metric" (at 116.5352 41.91 0)
       (effects (font (size 1.27 1.27)) hide)
     )
@@
       (effects (font (size 1.27 1.27)))
     )
-    (property "Footprint" "" (at 74.93 175.768 90)
+    (property "Footprint" "Resistor_SMD:R_0805_2012Metric" (at 74.93 175.768 90)
       (effects (font (size 1.27 1.27)) hide)
     )
@@
       (effects (font (size 1.27 1.27)))
     )
-    (property "Footprint" "" (at 214.63 111.4552 0)
+    (property "Footprint" "Capacitor_SMD:C_0805_2012Metric" (at 214.63 111.4552 0)
       (effects (font (size 1.27 1.27)) hide)
     )
@@
       (effects (font (size 1.27 1.27)) (justify left))
     )
-    (property "Footprint" "" (at 245.872 123.19 90)
+    (property "Footprint" "Resistor_SMD:R_0805_2012Metric" (at 245.872 123.19 90)
       (effects (font (size 1.27 1.27)) hide)
     )
@@
       (effects (font (size 1.27 1.27)))
     )
-    (property "Footprint" "" (at 39.37 183.388 90)
+    (property "Footprint" "Resistor_SMD:R_0805_2012Metric" (at 39.37 183.388 90)
       (effects (font (size 1.27 1.27)) hide)
     )
@@
       (effects (font (size 1.27 1.27)))
     )
-    (property "Footprint" "" (at 106.68 60.198 90)
+    (property "Footprint" "Resistor_SMD:R_0805_2012Metric" (at 106.68 60.198 90)
       (effects (font (size 1.27 1.27)) hide)
     )
@@
       (effects (font (size 1.27 1.27)))
     )
-    (property "Footprint" "" (at 90.805 149.86 0)
+    (property "Footprint" "Package_TO_SOT_SMD:SOT-223-3_TabPin2" (at 90.805 149.86 0)
       (effects (font (size 1.27 1.27) italic) (justify left) hide)
     )
@@
       (effects (font (size 1.27 1.27)) (justify right))
     )
-    (property "Footprint" "" (at 82.55 175.26 0)
+    (property "Footprint" "LED_SMD:LED_0805_2012Metric" (at 82.55 175.26 0)
       (effects (font (size 1.27 1.27)) hide)
     )
@@
       (effects (font (size 1.27 1.27)) (justify right))
     )
-    (property "Footprint" "" (at 223.52 143.51 0)
+    (property "Footprint" "Crystal:Crystal_SMD_MicroCrystal_CM9V-T1A-2Pin_1.6x1.0mm" (at 223.52 143.51 0)
       (effects (font (size 1.27 1.27)) hide)
     )
@@
       (effects (font (size 1.27 1.27)) (justify left))
     )
-    (property "Footprint" "" (at 170.18 -2.54 0)
+    (property "Footprint" "RF_Module:HOPERF_RFM9XW_SMD" (at 170.18 -2.54 0)
       (effects (font (size 1.27 1.27)) hide)
     )
@@
       (effects (font (size 1.27 1.27)))
     )
-    (property "Footprint" "" (at 92.71 59.69 0)
+    (property "Footprint" "Button_Switch_SMD:Panasonic_EVQPUL_EVQPUC" (at 92.71 59.69 0)
       (effects (font (size 1.27 1.27)) hide)
     )
@@
       (effects (font (size 1.27 1.27)) (justify right))
     )
-    (property "Footprint" "" (at 266.7 104.14 0)
+    (property "Footprint" "Connector_USB:USB_C_Receptacle_JAE_DX07S016JA1R1500" (at 266.7 104.14 0)
       (effects (font (size 1.27 1.27)) hide)
     )
@@
       (effects (font (size 1.27 1.27)) (justify left))
     )
-    (property "Footprint" "" (at 67.0052 148.59 0)
+    (property "Footprint" "Capacitor_SMD:C_0805_2012Metric" (at 67.0052 148.59 0)
       (effects (font (size 1.27 1.27)) hide)
     )
@@
       (effects (font (size 1.27 1.27)) (justify left))
     )
-    (property "Footprint" "" (at 127.9652 41.91 0)
+    (property "Footprint" "Capacitor_SMD:C_0805_2012Metric" (at 127.9652 41.91 0)
       (effects (font (size 1.27 1.27)) hide)
     )
@@
       (effects (font (size 1.27 1.27)))
     )
-    (property "Footprint" "" (at 231.14 146.3548 0)
+    (property "Footprint" "Capacitor_SMD:C_0805_2012Metric" (at 231.14 146.3548 0)
       (effects (font (size 1.27 1.27)) hide)
     )
@@
       (effects (font (size 1.27 1.27)))
     )
-    (property "Footprint" "" (at 39.37 177.292 90)
-      (effects (font (size 1.27 1.27)) hide)
-    )
+    (property "Footprint" "Resistor_SMD:R_0805_2012Metric" (at 39.37 177.292 90)
+      (effects (font (size 1.27 1.27)) hide)
+    )

Commit message: new placement and battery footprint
Parts:
- AE1: footprint (none) -> MountingHole:MountingHole_2.7mm_M2.5_DIN965_Pad_TopBottom
- BT1: footprint (none) -> Battery:BatteryHolder_Keystone_1060_1x2032
Changed lines of the file:
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@@
       (effects (font (size 1.27 1.27)) (justify left))
     )
-    (property "Footprint" "" (at 100.33 172.466 90)
+    (property "Footprint" "Battery:BatteryHolder_Keystone_1060_1x2032" (at 100.33 172.466 90)
       (effects (font (size 1.27 1.27)) hide)
     )
@@
       (effects (font (size 1.27 1.27)) (justify left))
     )
-    (property "Footprint" "" (at 278.13 25.4 0)
+    (property "Footprint" "MountingHole:MountingHole_2.7mm_M2.5_DIN965_Pad_TopBottom" (at 278.13 25.4 0)
       (effects (font (size 1.27 1.27)) hide)
     )

Commit message: ground plane, routing, comp layout
Parts:
- removed SW1: SW_Push_SPDT, Button_Switch_SMD:Panasonic_EVQPUL_EVQPUC, symbol Switch:SW_Push_SPDT
- added SW1: SW_Push, Button_Switch_SMD:SW_Push_1P1T_XKB_TS-1187A, symbol Switch:SW_Push
Connections:
- net EN: now also SW1.2
- net GND: now also SW1.1
Changed lines of the file:
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@@
     (stroke (width 0) (type default))
   )
-  (wire (pts (xy 87.63 64.77) (xy 87.63 59.69))
+  (wire (pts (xy 87.63 64.77) (xy 87.63 62.23))
     (stroke (width 0) (type default))
   )
@@
     )
   )
+  (symbol (lib_id "Switch:SW_Push") (at 92.71 62.23 0) (unit 1)
+    (in_bom yes) (on_board yes) (dnp no) (fields_autoplaced)
+    (property "Reference" "SW1" (at 92.71 54.61 0)
+      (effects (font (size 1.27 1.27)))
+    )
+    (property "Value" "SW_Push" (at 92.71 57.15 0)
+      (effects (font (size 1.27 1.27)))
+    )
+    (property "Footprint" "Button_Switch_SMD:SW_Push_1P1T_XKB_TS-1187A" (at 92.71 57.15 0)
+      (effects (font (size 1.27 1.27)) hide)
+    )
+    (property "Datasheet" "~" (at 92.71 57.15 0)
+      (effects (font (size 1.27 1.27)) hide)
+    )
+    (pin "1")
+    (pin "2")
+    (instances
+      (project "moirePCB"
+        (path "/527e949b-eaeb-4cf3-9920-57a6631a4ccb"
+          (reference "SW1") (unit 1)
+        )
+      )
+    )
+  )
   (symbol (lib_id "Device:Crystal") (at 223.52 143.51 90) (unit 1)
     (in_bom yes) (on_board yes) (dnp no)
@@
         )
       )
-    )
-  )
-  (symbol (lib_id "Switch:SW_Push_SPDT") (at 92.71 59.69 0) (unit 1)
-    (in_bom yes) (on_board yes) (dnp no) (fields_autoplaced)
-    (property "Reference" "SW1" (at 92.71 52.07 0)
-      (effects (font (size 1.27 1.27)))
-    )
-    (property "Value" "SW_Push_SPDT" (at 92.71 54.61 0)
-      (effects (font (size 1.27 1.27)))
-    )
-    (property "Footprint" "Button_Switch_SMD:Panasonic_EVQPUL_EVQPUC" (at 92.71 59.69 0)
-      (effects (font (size 1.27 1.27)) hide)
-    )
-    (property "Datasheet" "~" (at 92.71 59.69 0)
-      (effects (font (size 1.27 1.27)) hide)
-    )
-    (pin "1")
-    (pin "2")
-    (pin "3")
-    (instances
-      (project "moirePCB"
-        (path "/527e949b-eaeb-4cf3-9920-57a6631a4ccb"
-          (reference "SW1") (unit 1)
-        )
-      )

Commit message: pcb1 routing
Parts:
- added J2: Conn_01x12_Pin, Connector_PinHeader_2.54mm:PinHeader_1x12_P2.54mm_Vertical, symbol Connector:Conn_01x12_Pin
- SC1: footprint LED_SMD:LED_0805_2012Metric -> Connector_PinHeader_2.54mm:PinHeader_1x02_P2.54mm_Vertical
- renumbered D2 to CHG1, D1 to PGOOD1
Connections:
- net GPIO_34: now reaches U1.10 (IO34)
- net GPIO_34: now also J2.11 (Pin_11)
- net GPIO_35: now reaches U1.11 (IO35)
- net GPIO_35: now also J2.12 (Pin_12)
- net GPIO_25: now reaches U1.14 (IO25)
- net GPIO_25: now also J2.8 (Pin_8)
- net GPIO_26: now reaches U1.15 (IO26)
- net GPIO_26: now also J2.9 (Pin_9)
- net GPIO_27: now reaches U1.16 (IO27)
- net GPIO_27: now also J2.10 (Pin_10)
- net GPIO_14: now reaches U1.17 (IO14)
- net GPIO_14: now also U4.6 (RESET)
- net GPIO_12: now reaches U1.18 (IO12)
- net GPIO_12: now also U4.15 (DIO1)
- net GPIO_13: now reaches U1.20 (IO13)
- net GPIO_13: now also U4.14 (DIO0)
- net GPIO_15: now reaches U1.21 (IO15)
- net GPIO_15: now also J2.5 (Pin_5)
- net GPIO_2: now reaches U1.22 (IO2)
- net GPIO_2: now also J2.1 (Pin_1)
- net GPIO_4: now reaches U1.24 (IO4)
- net GPIO_4: now also J2.2 (Pin_2)
- net GPIO_9: now reaches U1.28 (SD2/IO9)
- net GPIO_9: now also J2.3 (Pin_3)
- net GPIO_10: now reaches U1.29 (SD3/IO10)
- net GPIO_10: now also J2.4 (Pin_4)
- net GPIO_5: now reaches U1.34 (IO5)
- net GPIO_5: now also U4.5 (NSS)
- net GPIO_18: now reaches U1.35 (IO18)
- net GPIO_18: now also U4.4 (SCK)
- net GPIO_23: now reaches U1.36 (IO23)
- net GPIO_23: now also U4.3 (MOSI)
- net GPIO_19: now reaches U1.38 (IO19)
- net GPIO_19: now also U4.2 (MISO)
- net GPIO_22: now reaches U1.39 (IO22)
- net GPIO_22: now also J2.7 (Pin_7)
- net GPIO_21: now reaches U1.42 (IO21)
- net GPIO_21: now also J2.6 (Pin_6)
