File: moirePCB/moirePCB.kicad_sch (KiCad schematic)
At the start: 55 parts, among them J1 USB_C_Receptacle, U1 ESP32-PICO-D4, U1 TLC555xD, U10 TLV73333PDBV, U2 BQ25504, U3 TLV73333PDBV, U4 RFM95W-915S2, U5 CH340E, U7 HDC1080, U8 AP2281-1WG-7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

Commit message: PCB 4: Silkscreen, part #s
Parts:
- BOOT1, EN1: LCSC Part # (none) -> C692460
- BT1: LCSC C173752 -> (none); LCSC Part # (none) -> C173752
- C1, C_FLTR1: LCSC Part # (none) -> C49678
- C2: LCSC Part # (none) -> C1710
- C2, C6: LCSC Part # (none) -> C1792
- C3: LCSC Part # (none) -> C128805
- C5: LCSC Part # (none) -> C15850
- C7: LCSC Part # (none) -> C282732
- C_HVR1, C_STOR1: LCSC Part # (none) -> C1779
- LDR1, SC1: LCSC Part # (none) -> C2883679
- R1: LCSC Part # (none) -> C2930231
- R10: LCSC Part # (none) -> C3016830
- R2: LCSC Part # (none) -> C17514
- R4: LCSC Part # (none) -> C352236
- R6: LCSC Part # (none) -> C27834
- R7: LCSC Part # (none) -> C218704
- R_OC+10: LCSC Part # (none) -> C843972
- R_OC_1: LCSC Part # (none) -> C422721
- R_OC_2: LCSC C422734 -> (none); LCSC Part # (none) -> C422734
- R_OK_1: LCSC Part # (none) -> C3000526
- R_OK_2, R_UV_2: LCSC Part # (none) -> C422717
- R_OK_3: LCSC Part # (none) -> C290129
- R_OV_1: LCSC Part # (none) -> C407395
- R_OV_2: LCSC Part # (none) -> C422723
- R_UV_1: LCSC Part # (none) -> C483106
- U1: LCSC Part # (none) -> C193707
- U1: LCSC C6987 -> (none); LCSC Part # (none) -> C6987
- U10, U3: LCSC Part # (none) -> C134139
- U2: LCSC Part # (none) -> C157471
- U4: LCSC C2844472 -> (none); LCSC Part # (none) -> C2844472
- U5: LCSC Part # (none) -> C99652
- U7: LCSC Part # (none) -> C82227
- U8, U9: LCSC Part # (none) -> C127279
- USB//OFF1, USB//SOLAR1: LCSC Part # (none) -> C431541
- Y2: LCSC Part # (none) -> C398713
Changed lines of the file:
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@@
+      (effects (font (size 1.27 1.27)) hide)
+    )
+    (property "LCSC Part #" "C127279" (at 114.3 167.64 0)
       (effects (font (size 1.27 1.27)) hide)
     )
@@
       (effects (font (size 1.27 1.27)) hide)
     )
+    (property "LCSC Part #" "C692460" (at 195.58 67.31 0)
+      (effects (font (size 1.27 1.27)) hide)
+    )
     (pin "1")
     (pin "2")
@@
     )
     (property "Datasheet" "http://www.ti.com/lit/ds/symlink/tlv733p.pdf" (at 31.75 113.03 0)
+      (effects (font (size 1.27 1.27)) hide)
+    )
+    (property "LCSC Part #" "C134139" (at 31.75 113.03 0)
       (effects (font (size 1.27 1.27)) hide)
     )
@@
     )
     (property "Datasheet" "http://www.ti.com/lit/ds/symlink/bq25504.pdf" (at 50.8 140.97 0)
+      (effects (font (size 1.27 1.27)) hide)
+    )
+    (property "LCSC Part #" "C157471" (at 58.42 161.29 0)
       (effects (font (size 1.27 1.27)) hide)
     )
@@
       (effects (font (size 1.27 1.27)) hide)
     )
-    (property "LCSC" "C173752" (at 100.33 173.99 0)
+    (property "LCSC Part #" "C173752" (at 100.33 173.99 0)
       (effects (font (size 1.27 1.27)) hide)
     )
@@
     )
     (property "Datasheet" "~" (at 62.23 67.31 0)
+      (effects (font (size 1.27 1.27)) hide)
+    )
+    (property "LCSC Part #" "C2930231" (at 62.23 67.31 0)
       (effects (font (size 1.27 1.27)) hide)
     )
@@
       (effects (font (size 1.27 1.27)) hide)
     )
+    (property "LCSC Part #" "C407395" (at 21.59 133.35 90)
+      (effects (font (size 1.27 1.27)) hide)
+    )
     (pin "1")
     (pin "2")
@@
       (effects (font (size 1.27 1.27)) hide)
     )
+    (property "LCSC Part #" "C218704" (at 128.27 166.37 90)
+      (effects (font (size 1.27 1.27)) hide)
+    )
     (pin "1")
     (pin "2")
@@
     )
     (property "Datasheet" "~" (at 224.79 115.57 0)
+      (effects (font (size 1.27 1.27)) hide)
+    )
+    (property "LCSC Part #" "C431541" (at 224.79 115.57 0)
       (effects (font (size 1.27 1.27)) hide)
     )
@@
       (effects (font (size 1.27 1.27)) hide)
     )
+    (property "LCSC Part #" "C1710" (at 21.59 90.17 0)
+      (effects (font (size 1.27 1.27)) hide)
+    )
     (pin "1")
     (pin "2")
@@
       (effects (font (size 1.27 1.27)) hide)
     )
+    (property "LCSC Part #" "C1792" (at 227.33 139.7 90)
+      (effects (font (size 1.27 1.27)) hide)
+    )
     (pin "1")
     (pin "2")
@@
       (effects (font (size 1.27 1.27)) hide)
     )
+    (property "LCSC Part #" "C1779" (at 81.28 172.72 90)
+      (effects (font (size 1.27 1.27)) hide)
+    )
     (pin "1")
     (pin "2")
@@
       (effects (font (size 1.27 1.27)) hide)
     )
+    (property "LCSC Part #" "C1779" (at 59.69 116.84 0)
+      (effects (font (size 1.27 1.27)) hide)
+    )
     (pin "1")
     (pin "2")
@@
       (effects (font (size 1.27 1.27)) hide)
     )
+    (property "LCSC Part #" "C15850" (at 115.57 38.1 0)
+      (effects (font (size 1.27 1.27)) hide)
+    )
     (pin "1")
     (pin "2")
@@
     )
     (property "Datasheet" "~" (at 29.21 133.35 0)
+      (effects (font (size 1.27 1.27)) hide)
+    )
+    (property "LCSC Part #" "C422723" (at 29.21 133.35 90)
       (effects (font (size 1.27 1.27)) hide)
     )
@@
       (effects (font (size 1.27 1.27)) hide)
     )
+    (property "LCSC Part #" "C282732" (at 217.17 110.49 90)
+      (effects (font (size 1.27 1.27)) hide)
+    )
     (pin "1")
     (pin "2")
@@
     )
     (property "Datasheet" "https://www.mpja.com/download/35227cpdata.pdf" (at 231.14 111.76 0)
+      (effects (font (size 1.27 1.27)) hide)
+    )
+    (property "LCSC Part #" "C99652" (at 222.25 91.44 0)
       (effects (font (size 1.27 1.27)) hide)
     )
@@
       (effects (font (size 1.27 1.27)) hide)
     )
+    (property "LCSC Part #" "C27834" (at 247.65 123.19 0)
+      (effects (font (size 1.27 1.27)) hide)
+    )
     (pin "1")
     (pin "2")
@@
     )
     (property "Datasheet" "~" (at 81.28 166.37 0)
+      (effects (font (size 1.27 1.27)) hide)
+    )
+    (property "LCSC Part #" "C49678" (at 81.28 166.37 90)
       (effects (font (size 1.27 1.27)) hide)
     )
@@
       (effects (font (size 1.27 1.27)) hide)
     )
+    (property "LCSC Part #" "C843972" (at 48.26 128.27 0)
+      (effects (font (size 1.27 1.27)) hide)
+    )
     (pin "1")
     (pin "2")
@@
       (effects (font (size 1.27 1.27)) hide)
     )
+    (property "LCSC Part #" "C352236" (at 138.43 181.61 0)
+      (effects (font (size 1.27 1.27)) hide)
+    )
     (pin "1")
     (pin "2")
@@
       (effects (font (size 1.27 1.27)) hide)
     )
+    (property "LCSC Part #" "C3016830" (at 110.49 91.44 90)
+      (effects (font (size 1.27 1.27)) hide)
+    )
     (pin "1")
     (pin "2")
@@
     )
     (property "Datasheet" "https://www.espressif.com/sites/default/files/documentation/esp32-pico-d4_datasheet_en.pdf" (at 160.02 123.19 0)
+      (effects (font (size 1.27 1.27)) hide)
+    )
+    (property "LCSC Part #" "C193707" (at 153.67 97.79 0)
       (effects (font (size 1.27 1.27)) hide)
     )
@@
       (effects (font (size 1.27 1.27)) hide)
     )
-    (property "LCSC" "C422734" (at 48.26 135.89 0)
+    (property "LCSC Part #" "C422734" (at 48.26 135.89 0)
       (effects (font (size 1.27 1.27)) hide)
     )
@@
     )
     (property "Datasheet" "~" (at 53.34 127 0)
+      (effects (font (size 1.27 1.27)) hide)
+    )
+    (property "LCSC Part #" "C431541" (at 53.34 127 0)
       (effects (font (size 1.27 1.27)) hide)
     )
@@
       (effects (font (size 1.27 1.27)) hide)
     )
+    (property "LCSC Part #" "C49678" (at 80.01 60.96 0)
+      (effects (font (size 1.27 1.27)) hide)
+    )
     (pin "1")
     (pin "2")
@@
       (effects (font (size 1.27 1.27)) hide)
     )
+    (property "LCSC Part #" "C692460" (at 119.38 62.23 0)
+      (effects (font (size 1.27 1.27)) hide)
+    )
     (pin "1")
     (pin "2")
@@
     )
     (property "Datasheet" "https://www.diodes.com/assets/Datasheets/AP2161.pdf" (at 100.33 113.03 0)
+      (effects (font (size 1.27 1.27)) hide)
+    )
+    (property "LCSC Part #" "C127279" (at 100.33 114.3 0)
       (effects (font (size 1.27 1.27)) hide)
     )
@@
       (effects (font (size 1.27 1.27)) hide)
     )
+    (property "LCSC Part #" "C398713" (at 223.52 143.51 90)
+      (effects (font (size 1.27 1.27)) hide)
+    )
     (pin "1")
     (pin "2")
@@
       (effects (font (size 1.27 1.27)) hide)
     )
-    (property "LCSC" "C6987" (at 46.99 80.01 0)
+    (property "LCSC Part #" "C6987" (at 46.99 80.01 0)
       (effects (font (size 1.27 1.27)) hide)
     )
@@
       (effects (font (size 1.27 1.27)) hide)
     )
+    (property "LCSC Part #" "C82227" (at 34.29 26.67 90)
+      (effects (font (size 1.27 1.27)) hide)
+    )
     (pin "1")
     (pin "2")
@@
       (effects (font (size 1.27 1.27)) hide)
     )
+    (property "LCSC Part #" "C17514" (at 67.31 80.01 90)
+      (effects (font (size 1.27 1.27)) hide)
+    )
     (pin "1")
     (pin "2")
@@
       (effects (font (size 1.27 1.27)))
     )
-    (property "LCSC" "C2844472" (at 254 39.37 0)
+    (property "LCSC Part #" "C2844472" (at 254 39.37 0)
       (effects (font (size 1.27 1.27)) hide)
     )
@@
       (effects (font (size 1.27 1.27)) hide)
     )
+    (property "LCSC Part #" "C3000526" (at 12.7 166.37 90)
+      (effects (font (size 1.27 1.27)) hide)
+    )
     (pin "1")
     (pin "2")
@@
       (effects (font (size 1.27 1.27)) hide)
     )
+    (property "LCSC Part #" "C290129" (at 19.05 154.94 0)
+      (effects (font (size 1.27 1.27)) hide)
+    )
     (pin "1")
     (pin "2")
@@
       (effects (font (size 1.27 1.27)) hide)
     )
+    (property "LCSC Part #" "C2883679" (at 67.31 115.57 0)
+      (effects (font (size 1.27 1.27)) hide)
+    )
     (pin "1")
     (pin "2")
@@
     )
     (property "Datasheet" "~" (at 15.24 138.43 0)
+      (effects (font (size 1.27 1.27)) hide)
+    )
+    (property "LCSC Part #" "C483106" (at 15.24 138.43 0)
       (effects (font (size 1.27 1.27)) hide)
     )
@@
       (effects (font (size 1.27 1.27)) hide)
     )
+    (property "LCSC Part #" "C422717" (at 19.05 162.56 0)
+      (effects (font (size 1.27 1.27)) hide)
+    )
     (pin "1")
     (pin "2")
@@
     )
     (property "Datasheet" "~" (at 127 38.1 0)
+      (effects (font (size 1.27 1.27)) hide)
+    )
+    (property "LCSC Part #" "C49678" (at 127 38.1 0)
       (effects (font (size 1.27 1.27)) hide)
     )
@@
     )
     (property "Datasheet" "http://www.ti.com/lit/ds/symlink/tlv733p.pdf" (at 78.74 191.77 0)
+      (effects (font (size 1.27 1.27)) hide)
+    )
+    (property "LCSC Part #" "C134139" (at 78.74 191.77 0)
       (effects (font (size 1.27 1.27)) hide)
     )
@@
       (effects (font (size 1.27 1.27)) hide)
     )
+    (property "LCSC Part #" "C422717" (at 15.24 146.05 0)
+      (effects (font (size 1.27 1.27)) hide)
+    )
     (pin "1")
     (pin "2")
@@
     )
     (property "Datasheet" "~" (at 30.48 177.8 0)
+      (effects (font (size 1.27 1.27)) hide)
+    )
+    (property "LCSC Part #" "C128805" (at 30.48 177.8 90)
       (effects (font (size 1.27 1.27)) hide)
     )
@@
       (effects (font (size 1.27 1.27)) hide)
     )
+    (property "LCSC Part #" "C2883679" (at 97.79 91.44 90)
+      (effects (font (size 1.27 1.27)) hide)
+    )
     (pin "1")
     (pin "2")
@@
       (effects (font (size 1.27 1.27)) hide)
     )
+    (property "LCSC Part #" "C422721" (at 41.91 120.65 0)
+      (effects (font (size 1.27 1.27)) hide)
+    )
     (pin "1")
     (pin "2")
@@
       (effects (font (size 1.27 1.27)) hide)
     )
+    (property "LCSC Part #" "C1792" (at 227.33 147.32 90)
+      (effects (font (size 1.27 1.27)) hide)
+    )

Commit message: pcb4: replace rfm95 with correct freq
Parts:
- U4: LCSC Part # C2844472 -> C2844473
Changed lines of the file:
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@@
       (effects (font (size 1.27 1.27)))
     )
-    (property "LCSC Part #" "C2844472" (at 254 39.37 0)
+    (property "LCSC Part #" "C2844473" (at 254 39.37 0)
       (effects (font (size 1.27 1.27)) hide)
     )
