File: moirePCB/moirePCB.kicad_pcb (KiCad board)
At the start: 2 copper layers, 37 parts, among them J1 USB_C_Receptacle, J2 Conn_01x12_Pin, SW1 SW_Push, SW3 SW_DPDT_x2, U1 ESP32-PICO-D4, U2 BQ24075RGT, U3 UA78M33, U4 RFM95W-915S2, U5 CH340E, U6 TLC555xD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

Commit message: routing wip
Parts:
- moved U6 104.4 mm to (66.6, 117.0), turned to 90 degrees
- moved R5 98.2 mm to (71.3, 114.6), turned to 90 degrees
- moved C8 97.4 mm to (71.3, 119.0), turned to 90 degrees
- moved R8 94.1 mm to (74.2, 114.6), turned to 90 degrees
- moved C9 93.2 mm to (74.3, 119.0), turned to 90 degrees
- moved J2 70.6 mm to (53.2, 34.3)
- moved GND1 52.0 mm to (52.9, 68.9), turned to 0 degrees
- moved CLK1 44.4 mm to (57.2, 81.8), turned to 0 degrees
- moved VCC1 42.2 mm to (52.9, 80.7), turned to 0 degrees
- moved U3 28.7 mm to (67.7, 85.9), turned to 180 degrees
- moved R4 18.7 mm to (81.2, 39.4), turned to 180 degrees
- moved U1 8.41 mm to (67.2, 71.7)
- moved U5 7.48 mm to (65.3, 58.1), turned to -90 degrees
- moved R2 6.55 mm to (79.7, 73.0), turned to 180 degrees
- moved R3 6.01 mm to (76.4, 76.8)
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Routing:
- added copper zone on In2.Cu, net GND
Other:
- board outline added: 38.8 x 200.6 mm
- copper layers 2 -> 4

Commit message: maddie call
Parts:
- moved C4 24.8 mm to (61.8, 82.2), turned to 0 degrees
- moved CHG1 21.7 mm to (61.8, 87.2), turned to 180 degrees
- moved C3 20.7 mm to (67.4, 82.3), turned to 0 degrees
- moved U3 17.4 mm to (84.5, 90.2), turned to -90 degrees
- moved PGOOD1 16.5 mm to (67.3, 87.4), turned to 0 degrees
- moved Y2 14.8 mm to (59.6, 77.8), turned to 90 degrees
- moved C2 14.3 mm to (56.9, 76.8), turned to 0 degrees
- moved C6 13.1 mm to (56.9, 78.8), turned to 180 degrees
- moved R6 13.0 mm to (77.2, 54.3), turned to 180 degrees
- moved CLK1 11.0 mm to (52.8, 91.9)
- moved R2 10.4 mm to (77.1, 62.9)
- moved R7 5.45 mm to (77.2, 58.5), turned to 0 degrees
- moved R1 5.16 mm to (81.7, 71.8)
- moved U1 3.29 mm to (65.8, 68.7)
- moved R3 2.58 mm to (75.7, 74.4)
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Routing:
- net VCC: track 108.6 -> 330.0 mm, vias 0 -> 4
- net GND: track 203.2 -> 294.3 mm, vias 0 -> 32
- net /GPIO_18: track 0.00 -> 68.7 mm, vias 0 -> 1
- net /EN: track 0.00 -> 67.3 mm
- net /GPIO_15: track 0.00 -> 49.5 mm, vias 0 -> 1
- net /GPIO_2: track 0.00 -> 48.7 mm, vias 0 -> 2
- net /GPIO_4: track 0.00 -> 44.9 mm, vias 0 -> 1
- net /GPIO_14: track 0.00 -> 42.5 mm, vias 0 -> 2
- net Net-(ONOFF1A-B): track 0.00 -> 41.9 mm, vias 0 -> 2
- net Net-(CHG1-A): track 0.00 -> 40.3 mm, vias 0 -> 2
- net /GPIO_12: track 0.00 -> 40.0 mm, vias 0 -> 2
- net /GPIO_9: track 0.00 -> 39.6 mm, vias 0 -> 1
- net /GPIO_25: track 0.00 -> 36.5 mm, vias 0 -> 1
- net /GPIO_13: track 0.00 -> 36.3 mm, vias 0 -> 2
- net /GPIO_10: track 0.00 -> 35.6 mm, vias 0 -> 1
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Other:
- board size 38.8 x 200.6 mm -> 39.8 x 200.6 mm
